Commit message: navigation working

File: src/diff_drive_robot/urdf/diff_drive.robot_control.xacro (robot description, xacro)
@@ -3,5 +3,6 @@
     <ros2_control name="DiffDriveRobotHardwareInterface" type="system">
         <hardware>
-            <plugin>mock_components/GenericSystem</plugin>
+            <!-- <plugin>mock_components/GenericSystem</plugin> -->
+            <plugin>gz_ros2_control/GazeboSimSystem</plugin>
             <param name="calculate_dynamics">true</param>
         </hardware>

File: src/diff_drive_robot/urdf/diff_drive.urdf.xacro (robot description, xacro)
@@ -1,108 +1,7 @@
 <?xml version="1.0"?>
 <robot xmlns:xacro="http://www.ros.org/wiki/xacro" name="diff_drive">
-    <xacro:include filename="xacros/robot_paras.xacro" />
-    <xacro:include filename="xacros/colors.xacro" />
-    <xacro:include filename="diff_drive.robot_control.xacro" />
-    <link name="base_link">
-    </link>
-    <joint name="base_to_body" type="fixed">
-        <parent link="base_link" />
-        <child link="body_link" />
-        <origin xyz="0 0 ${body_box_size_z/2}" rpy="0 0 ${-pi/2}" />
-        <axis xyz="0 0 0" />
-    </joint>
-    <link name="body_link">
-        <visual>
-            <geometry>
-                <box size="${body_box_size_x} ${body_box_size_y} ${body_box_size_z}" />
-            </geometry>
-            <material name="orange" />
-            <origin xyz="0 0 0" rpy="0 0 0" />
-        </visual>
-        <collision>
-            <geometry>
-                <box size="${body_box_size_x} ${body_box_size_y} ${body_box_size_z}" />
-            </geometry>
-            <origin xyz="0 0 ${body_box_size_z/2}" rpy="0 0 0" />
-        </collision>
-        <inertial>
-            <mass value="2.0" />
-            <inertia ixx="0.1" ixy="0.0" ixz="0.0" iyy="0.1" iyz="0.0" izz="0.1" />
-        </inertial>
-    </link>
-    <joint name="body_to_lw" type="continuous">
-        <parent link="body_link" />
-        <child link="left_wheel_link" />
-        <origin xyz="${body_box_size_x/2 + wheel_offset} 0 ${-body_box_size_z/2}" rpy="0 ${pi/2} 0" />
-        <axis xyz="0 0 1" />
-    </joint>
-    <link name="left_wheel_link">
-        <visual>
-            <geometry>
-                <cylinder radius="${wheel_radius}" length="${wheel_length}" />
-            </geometry>
-            <material name="blue" />
-            <origin xyz="0 0 0" rpy="0 0 0" />
-        </visual>
-        <collision>
-            <geometry>
-                <cylinder radius="${wheel_radius}" length="${wheel_length}" />
-            </geometry>
-            <origin xyz="0 0 0" rpy="0 0 0" />
-        </collision>
-        <inertial>
-            <mass value="2.0" />
-            <inertia ixx="0.1" ixy="0.0" ixz="0.0" iyy="0.1" iyz="0.0" izz="0.1" />
-        </inertial>
-    </link>
-    <joint name="body_to_rw" type="continuous">
-        <parent link="body_link" />
-        <child link="right_wheel_link" />
-        <origin xyz="${-body_box_size_x/2 - wheel_offset} 0 ${-body_box_size_z/2}" rpy="0 ${-pi/2} 0" />
-        <axis xyz="0 0 -1" />
-    </joint>
-    <link name="right_wheel_link">
-        <visual>
-            <geometry>
-                <cylinder radius="${wheel_radius}" length="${wheel_length}" />
-            </geometry>
-            <material name="blue" />
-            <origin xyz="0 0 0" rpy="0 0 0" />
-        </visual>
-        <collision>
-            <geometry>
-                <cylinder radius="${wheel_radius}" length="${wheel_length}" />
-            </geometry>
-            <origin xyz="0 0 0" rpy="0 0 0" />
-        </collision>
-        <inertial>
-            <mass value="2.0" />
-            <inertia ixx="0.1" ixy="0.0" ixz="0.0" iyy="0.1" iyz="0.0" izz="0.1" />
-        </inertial>
-    </link>
-    <joint name="body_to_caster_wheel_link" type="fixed">
-        <parent link="body_link" />
-        <child link="caster_wheel_link" />
-        <origin xyz="0 ${-body_box_size_y/2 + wheel_radius} ${-body_box_size_z/2}" rpy="0 0 0" />
-        <axis xyz="0 0 0" />
-    </joint>
-    <link name="caster_wheel_link">
-        <visual>
-            <geometry>
-                <sphere radius="${wheel_radius}" />
-            </geometry>
-            <material name="blue" />
-            <origin xyz="0 0 0" rpy="0 0 0" />
-        </visual>
-        <collision>
-            <geometry>
-                <sphere radius="${wheel_radius}" />
-            </geometry>
-            <origin xyz="0 0 0" rpy="0 0 0" />
-        </collision>
-        <inertial>
-            <mass value="2.0" />
-            <inertia ixx="0.1" ixy="0.0" ixz="0.0" iyy="0.1" iyz="0.0" izz="0.1" />
-        </inertial>
-    </link>
+    <!-- <xacro:include filename="gazebo_control.xacro" /> -->
+    <xacro:include filename="robot.gazebo.xacro" />
+    <xacro:include filename="robot_core.urdf.xacro" />
+    <!-- <xacro:include filename="diff_drive.robot_control.xacro" /> -->
 </robot>

File: src/diff_drive_robot/urdf/xacros/robot_paras.xacro (robot description, xacro)
@@ -1,11 +1,14 @@
 <?xml version="1.0"?>
 <robot xmlns:xacro="http://www.ros.org/wiki/xacro">
-    <xacro:property name="wheel_offset" value="0.05"/>
+    <xacro:property name="wheel_offset" value="0.01" />
     <!-- body link -->
-    <xacro:property name="body_box_size_x" value="2.0"/>
-    <xacro:property name="body_box_size_y" value="3"/>
-    <xacro:property name="body_box_size_z" value="0.75"/>
+    <xacro:property name="body_box_size_x" value="0.5" />
+    <xacro:property name="body_box_size_y" value="0.6" />
+    <xacro:property name="body_box_size_z" value="0.1" />
     <!-- Wheel -->
-    <xacro:property name="wheel_radius" value="0.4"/>
-    <xacro:property name="wheel_length" value="0.1"/>
+    <xacro:property name="wheel_radius" value="0.08" />
+    <xacro:property name="wheel_length" value="0.04" />
+    <!-- Lidar -->
+    <xacro:property name="lidar_radius" value="0.06" />
+    <xacro:property name="lidar_length" value="0.04" />
 </robot>
